Commit message: Added the new ROS1 migration of the checkpoint 1 project

File: my_rb1_description/urdf/my_rb1_robot.urdf (robot description, URDF)
Before this commit: robot rb1_robot, 7 links, 6 joints
Links:
- link back_caster: mass 0.15 -> 0.5
- link base_link: mass 24 -> 20.5
- link front_caster: mass 0.15 -> 0.5
- link front_laser: mass 0.2 -> None; geometry 
- link left_wheel: mass 0.25 -> 1.5
- link right_wheel: mass 0.25 -> 1.5
Joints:
- joint base_link_front_laser_joint: origin xyz=0.25 0 0.075 rpy=0 0 0 -> xyz=0.25 0 0.075 rpy=3.14 0 0
- joint base_link_left_wheel_joint: limit effort=10000 velocity=1000 -> (none); origin xyz=0 -0.2 -0.15 rpy=0 0 0 -> xyz=0 0.2 -0.15 rpy=0 0 0
- joint base_link_right_wheel_joint: limit effort=10000 velocity=1000 -> (none); origin xyz=0 0.2 -0.15 rpy=0 0 0 -> xyz=0 -0.2 -0.15 rpy=0 0 0

Commit message: Update my_rb1_robot.urdf

File: my_rb1_description/urdf/my_rb1_robot.urdf (robot description, URDF)
Before this commit: robot rb1_robot, 7 links, 6 joints
Joints:
- joint base_link_front_laser_joint: origin xyz=0.25 0 0.075 rpy=3.14 0 0 -> xyz=0.25 0 0.075 rpy=0 0 0
